Commit message: add_hand

File: BBL_robot_description/urdf/BBL.urdf.xacro (robot description, xacro)
@@ -427,9 +427,60 @@
       friction="0.0" />
   </joint>
-  <link name="tool"/>
-  <joint name="tool_joint" type="fixed">
-     <origin xyz="0 0 0" rpy="0 0 0"/>
-     <parent link="link6"/>
-     <child link="tool"/>
+<!--  <link name="tool"/>-->
+<!--  <joint name="tool_joint" type="fixed">-->
+<!--     <origin xyz="0 0 0" rpy="0 0 0"/>-->
+<!--     <parent link="link6"/>-->
+<!--     <child link="tool"/>-->
+<!--  </joint>-->
+    <link
+    name="hand">
+    <inertial>
+      <origin
+        xyz="-1.4558E-07 -4.1668E-07 1.0004E-07"
+        rpy="0 0 0" />
+      <mass
+        value="0.35608" />
+      <inertia
+        ixx="0.0017195"
+        ixy="-5.3819E-06"
+        ixz="8.6395E-05"
+        iyy="0.0016178"
+        iyz="7.7129E-06"
+        izz="0.00041293" />
+    </inertial>
+    <visual>
+      <origin
+        xyz="-0.00468 -0.0815 0.00171"
+        rpy="0 0 0" />
+      <geometry>
+        <mesh
+          filename="package://BBL_robot_description/meshes/hand.STL" />
+      </geometry>
+      <material
+        name="">
+        <color
+          rgba="0.75294 0.75294 0.75294 1" />
+      </material>
+    </visual>
+    <collision>
+      <origin
+        xyz="0 0 0"
+        rpy="0 0 0" />
+      <geometry>
+        <mesh
+          filename="package://BBL_robot_description/meshes/hand.STL" />
+      </geometry>
+    </collision>
+  </link>
+    <joint
+    name="hand_joint"
+    type="fixed">
+    <origin
+      xyz="0 0 0"
+      rpy="-1.5708 0 0" />
+    <parent
+      link="link6" />
+    <child
+      link="hand" />
   </joint>
   <xacro:transmission_acro joint_name="joint1"/>
